File: docs/kicad/windTester/windBreadboard.kicad_pcb (KiCad board)
At the start: 2 copper layers, 19 parts, among them Q1 BC547, U1 LM324A

Commit message: played around again with idea of a windTester opAmp driven breadboard
Parts:
- added J1: Conn_01x01, 0_my_footprints:myPinHeader_1x01, F.Cu at (-54.7, 86.9)
- added J10: Conn_01x01, 0_my_footprints:myPinHeader_1x01, F.Cu at (-59.2, 94.2)
- added J2: Conn_01x01, 0_my_footprints:myPinHeader_1x01, F.Cu at (-58.3, 90.5)
- added J3: Conn_01x01, 0_my_footprints:myPinHeader_1x01, F.Cu at (-34.8, 68.2)
- added J4: Conn_01x01, 0_my_footprints:myPinHeader_1x01, F.Cu at (55.9, 55.9)
- added J5: Conn_01x01, 0_my_footprints:myPinHeader_1x01, F.Cu at (83.8, 76.2)
- added J6: Conn_01x01, 0_my_footprints:myPinHeader_1x01, F.Cu at (-66.5, 91.4)
- added J7: Conn_01x01, 0_my_footprints:myPinHeader_1x01, F.Cu at (34.3, 45.7)
- added J8: Conn_01x01, 0_my_footprints:myPinHeader_1x01, F.Cu at (101.6, 114.3)
- added J9: Conn_01x01, 0_my_footprints:myPinHeader_1x01, F.Cu at (-35.3, 57.2)
- moved R13 104.2 mm to (-27.9, 111.8), turned to 0 degrees
- moved Q1 104.0 mm to (-29.2, 120.7)
- moved R14 91.8 mm to (-19.1, 116.8), turned to 0 degrees
- moved C3 78.4 mm to (15.2, 55.9)
- moved R10 77.4 mm to (63.5, 114.3)
- moved R9 66.7 mm to (73.7, 121.9), turned to 90 degrees
- moved R11 62.0 mm to (71.1, 108.0), turned to 180 degrees
- moved R1 45.7 mm to (48.3, 45.7), turned to 180 degrees
- moved R12 43.2 mm to (83.8, 108.0)
- moved C1 40.6 mm to (50.8, 45.7)
- moved U1 20.9 mm to (78.7, 68.6)
- moved R2 20.3 mm to (61.0, 45.7), turned to 180 degrees
- moved R4 18.3 mm to (78.7, 45.7)
- moved R3 16.3 mm to (66.0, 38.1), turned to 270 degrees
- moved R8 16.1 mm to (76.2, 114.3), turned to 0 degrees
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Routing:
- net Net-(R4-Pad1): track 63.3 -> 22.9 mm, vias 6 -> 2
- net GND: track 86.4 -> 50.8 mm, vias 6 -> 0
- net Net-(R2-Pad1): track 22.9 -> 53.3 mm, vias 2 -> 6
- net +12V: track 35.6 -> 10.2 mm, vias 4 -> 0
- net Net-(R5-Pad1): track 10.2 -> 25.4 mm, vias 0 -> 2
- net SIGNALA: track 40.5 -> 27.9 mm, vias 4 -> 2
- net (no net): track 10.2 -> 0.00 mm
- added copper zone on F.Cu, net +12V
- added copper zone on B.Cu, net GND
